File: schematics_kicad/kicad/tentacle_daq_saleae.kicad_sch (KiCad schematic)
At the start: 5 parts, among them T901 tentacle, T902 tentacle, T903 tentacle

Commit message: Updating schematics for RPI_PICO_W for tentacle v0.4
Parts:
- T902: symbol 00_project_library:tentacle_gpio -> 00_project_library:tentacle_v03_gpio
Changed lines of the file:
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@@
 	(label "error_data1"
 		(at 130.81 127 0)
-		(fields_autoplaced yes)
 		(effects
 			(font
@@
 	(label "SIGNAL_TRIGGER2"
 		(at 74.93 66.04 0)
-		(fields_autoplaced yes)
 		(effects
 			(font
@@
 	(label "trigger1"
 		(at 130.81 116.84 0)
-		(fields_autoplaced yes)
 		(effects
 			(font
@@
 	(label "error_data2"
 		(at 130.81 132.08 0)
-		(fields_autoplaced yes)
 		(effects
 			(font
@@
 	(label "trigger2"
 		(at 130.81 121.92 0)
-		(fields_autoplaced yes)
 		(effects
 			(font
@@
 	(label "SIGNAL_DATA2"
 		(at 74.93 76.2 0)
-		(fields_autoplaced yes)
 		(effects
 			(font
@@
 	(label "SIGNAL_DATA1"
 		(at 74.93 71.12 0)
-		(fields_autoplaced yes)
 		(effects
 			(font
@@
 	(label "SIGNAL_TRIGGER1"
 		(at 74.93 60.96 0)
-		(fields_autoplaced yes)
 		(effects
 			(font
@@
 	)
 	(symbol
-		(lib_id "00_project_library:tentacle_gpio")
+		(lib_id "00_project_library:tentacle_v03_gpio")
 		(at 104.14 109.22 0)
 		(unit 1)
