File: schematics_kicad/kicad/tenacle_MCU_RPI_PICO.kicad_sch (KiCad schematic)
At the start: 3 parts, among them T201 tentacle_octobus, T202 tentacle_relay

Commit message: tmp2
Changed lines of the file:
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@@
 		)
 	)
-	(text_box "Serial resistor allows introducing errors by overriding the signal (see tentacle_daq_saleae)"
+	(text_box "Serial resistor allows introducing errors by overriding the signal\n(see tentacle_daq_saleae)\n"
 		(exclude_from_sim no)
-		(at 154.94 36.83 0)
-		(size 20.32 15.24)
+		(at 151.13 40.64 0)
+		(size 29.21 10.16)
 		(stroke
 			(width 0)
